File: ESP32-PDM-BASE.kicad_sch (KiCad schematic)
At the start: 11 parts, among them J1 Conn_02x06_Top_Bottom, U1 ESP32-S3-MINI-1

Commit message: unfinished work
Parts:
- added H1, H2: MountingHole, symbol Mechanical:MountingHole
Changed lines of the file:
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@@
 	(label "IO7"
 		(at 88.9 90.17 0)
-		(fields_autoplaced yes)
 		(effects
 			(font
@@
 	(label "IO4"
 		(at 104.14 48.26 180)
-		(fields_autoplaced yes)
 		(effects
 			(font
@@
 	(label "IO6"
 		(at 120.65 93.98 180)
-		(fields_autoplaced yes)
 		(effects
 			(font
@@
 	(label "SW_IN2"
 		(at 71.12 85.09 0)
-		(fields_autoplaced yes)
 		(effects
 			(font
@@
 	(label "IO8"
 		(at 88.9 105.41 0)
-		(fields_autoplaced yes)
 		(effects
 			(font
@@
 	(label "USB_TXD"
 		(at 154.94 76.2 0)
-		(fields_autoplaced yes)
 		(effects
 			(font
@@
 	(label "IO17"
 		(at 120.65 121.92 180)
-		(fields_autoplaced yes)
 		(effects
 			(font
@@
 	(label "IO12"
 		(at 120.65 109.22 180)
-		(fields_autoplaced yes)
 		(effects
 			(font
@@
 	(label "IO13"
 		(at 33.02 104.14 180)
-		(fields_autoplaced yes)
 		(effects
 			(font
@@
 	(label "IO13"
 		(at 120.65 111.76 180)
-		(fields_autoplaced yes)
 		(effects
 			(font
@@
 	(label "IO9"
 		(at 120.65 101.6 180)
-		(fields_autoplaced yes)
 		(effects
 			(font
@@
 	(label "EN"
 		(at 212.09 54.61 0)
-		(fields_autoplaced yes)
 		(effects
 			(font
@@
 	(label "IO18"
 		(at 184.15 78.74 180)
-		(fields_autoplaced yes)
 		(effects
 			(font
@@
 	(label "IO9"
 		(at 88.9 121.92 0)
-		(fields_autoplaced yes)
 		(effects
 			(font
@@
 	(label "IO2"
 		(at 120.65 83.82 180)
-		(fields_autoplaced yes)
 		(effects
 			(font
@@
 	(label "IO5"
 		(at 120.65 91.44 180)
-		(fields_autoplaced yes)
 		(effects
 			(font
@@
 	(label "IO7"
 		(at 120.65 96.52 180)
-		(fields_autoplaced yes)
 		(effects
 			(font
@@
 	(label "IO18"
 		(at 120.65 124.46 180)
-		(fields_autoplaced yes)
 		(effects
 			(font
@@
 	(label "SW_IN4"
 		(at 116.84 35.56 0)
-		(fields_autoplaced yes)
 		(effects
 			(font
@@
 	(label "SW_IN1"
 		(at 71.12 68.58 0)
-		(fields_autoplaced yes)
 		(effects
 			(font
@@
 	(label "IO10"
 		(at 120.65 104.14 180)
-		(fields_autoplaced yes)
 		(effects
 			(font
@@
 	(label "SW_IN4"
 		(at 71.12 116.84 0)
-		(fields_autoplaced yes)
 		(effects
 			(font
@@
 	(label "IO6"
 		(at 88.9 73.66 0)
-		(fields_autoplaced yes)
 		(effects
 			(font
@@
 	(label "IO8"
 		(at 120.65 99.06 180)
-		(fields_autoplaced yes)
 		(effects
 			(font
@@
 	(label "SW_IN3"
 		(at 104.14 45.72 180)
-		(fields_autoplaced yes)
 		(effects
 			(font
@@
 	(label "IO5"
 		(at 116.84 38.1 0)
-		(fields_autoplaced yes)
 		(effects
 			(font
@@
 	(label "IO10"
 		(at 33.02 92.71 180)
-		(fields_autoplaced yes)
 		(effects
 			(font
@@
 	(label "SW_IN2"
 		(at 104.14 40.64 180)
-		(fields_autoplaced yes)
 		(effects
 			(font
@@
 	(label "IO12"
 		(at 33.02 100.33 180)
-		(fields_autoplaced yes)
 		(effects
 			(font
@@
 	(label "IO3"
 		(at 120.65 86.36 180)
-		(fields_autoplaced yes)
 		(effects
 			(font
@@
 	(label "IO17"
 		(at 184.15 74.93 180)
-		(fields_autoplaced yes)
 		(effects
 			(font
@@
 	(label "IO0"
 		(at 212.09 50.8 0)
-		(fields_autoplaced yes)
 		(effects
 			(font
@@
 	(label "USB_RXD"
 		(at 154.94 73.66 0)
-		(fields_autoplaced yes)
 		(effects
 			(font
@@
 	(label "IO11"
 		(at 33.02 96.52 180)
-		(fields_autoplaced yes)
 		(effects
 			(font
@@
 	(label "USB_TXD"
 		(at 212.09 43.18 0)
-		(fields_autoplaced yes)
 		(effects
 			(font
@@
 	(label "EN"
 		(at 120.65 73.66 180)
-		(fields_autoplaced yes)
 		(effects
 			(font
@@
 	(label "IO3"
 		(at 104.14 43.18 180)
-		(fields_autoplaced yes)
 		(effects
 			(font
@@
 	(label "USB_RXD"
 		(at 212.09 46.99 0)
-		(fields_autoplaced yes)
 		(effects
 			(font
@@
 	(label "IO2"
 		(at 104.14 38.1 180)
-		(fields_autoplaced yes)
 		(effects
 			(font
@@
 	(label "IO0"
 		(at 120.65 78.74 180)
-		(fields_autoplaced yes)
 		(effects
 			(font
@@
 	(label "SW_IN1"
 		(at 104.14 35.56 180)
-		(fields_autoplaced yes)
 		(effects
 			(font
@@
 	(label "IO4"
 		(at 120.65 88.9 180)
-		(fields_autoplaced yes)
 		(effects
 			(font
@@
 	(label "IO11"
 		(at 120.65 106.68 180)
-		(fields_autoplaced yes)
 		(effects
 			(font
@@
 	(label "SW_IN3"
 		(at 71.12 100.33 0)
-		(fields_autoplaced yes)
 		(effects
 			(font
@@
 					(unit 1)
 				)
+			)
+		)
+	)
+	(symbol
+		(lib_id "Mechanical:MountingHole")
+		(at 186.69 134.62 0)
+		(unit 1)
+		(exclude_from_sim yes)
+		(in_bom no)
+		(on_board yes)
+		(dnp no)
+		(fields_autoplaced yes)
+		(property "Reference" "H1"
+			(at 189.23 133.3499 0)
+			(effects
+				(font
+					(size 1.27 1.27)
+				)
+				(justify left)
+			)
+		)
+		(property "Value" "MountingHole"
+			(at 189.23 135.8899 0)
+			(effects
+				(font
+					(size 1.27 1.27)
+				)
+				(justify left)
+			)
+		)
+		(property "Footprint" ""
+			(at 186.69 134.62 0)
+			(effects
+				(font
+					(size 1.27 1.27)
+				)
+				(hide yes)
+			)
+		)
+		(property "Datasheet" "~"
+			(at 186.69 134.62 0)
+			(effects
+				(font
+					(size 1.27 1.27)
+				)
+				(hide yes)
+			)
+		)
+		(property "Description" "Mounting Hole without connection"
+			(at 186.69 134.62 0)
+			(effects
+				(font
+					(size 1.27 1.27)
+				)
+				(hide yes)
+			)
+		)
+		(instances
+			(project ""
+				(path "/d0898527-243c-48e9-a217-df57be741056"
+					(reference "H1")
+					(unit 1)
+				)
+			)
+		)
+	)
+	(symbol
+		(lib_id "Mechanical:MountingHole")
+		(at 186.69 140.97 0)
+		(unit 1)
+		(exclude_from_sim yes)
+		(in_bom no)
+		(on_board yes)
+		(dnp no)
+		(fields_autoplaced yes)
+		(property "Reference" "H2"
+			(at 189.23 139.6999 0)
+			(effects
+				(font
+					(size 1.27 1.27)
+				)
+				(justify left)
+			)
+		)
+		(property "Value" "MountingHole"
+			(at 189.23 142.2399 0)
+			(effects
+				(font
+					(size 1.27 1.27)
+				)
+				(justify left)
+			)
+		)
+		(property "Footprint" ""
+			(at 186.69 140.97 0)
+			(effects
+				(font
+					(size 1.27 1.27)
+				)
+				(hide yes)
+			)
+		)
+		(property "Datasheet" "~"
+			(at 186.69 140.97 0)
+			(effects
+				(font
+					(size 1.27 1.27)
+				)
+				(hide yes)
+			)
+		)
+		(property "Description" "Mounting Hole without connection"
+			(at 186.69 140.97 0)
+			(effects
+				(font
+					(size 1.27 1.27)
+				)
+				(hide yes)
+			)
+		)
+		(instances
+			(project ""
+				(path "/d0898527-243c-48e9-a217-df57be741056"
+					(reference "H2")
+					(unit 1)
+				)
