File: can.kicad_sch (KiCad schematic)
At the start: 12 parts, among them J4 Conn_01x04, U5 ISO1044, U6 TPS7B91050

Commit message: Apply JLCPCB BOM audit fixes and add module ID / switch sense
- Remove CH340C and auto-reset circuit; USB-C goes to native USB
  (IO19 = D-, IO20 = D+). UART0 left unconnected.
- USB-C: HRO TYPE-C-31-M-12 (shell pins renumbered SH to match footprint).
- F1/F3: 1812L050/60GR (60 V, 500 mA hold); old part was rated 30 V max.
- D2/D3/D11: DSK16 (60 V) replacing out-of-stock DSS14U.
- D9: PESD2CAN replacing unavailable ESDCAN01-2BWY (SOT-23).
- L1: SWPA6045S8R2MT (Isat 3.9 A > LMR51610 peak limit 1.95 A).
- Feedback divider 68k/22k (basic parts): Vout 3.27 V with Vref 0.8 V.
- Basic-library swaps: TS-1187A buttons, 0805 2.2uF/50V, 49.9 R,
  BC817-40.
- Move the ST pull-ups to the output module.
- Header pin 12 becomes MOD_ID (IO1, 10k pull-up).
- SW1-SW4 to IO14/IO15/IO16/IO21 with 10k pull-downs, so the firmware
  can read the physical switches.
- Add LCSC part numbers for changed parts and main ICs.

ERC: 38 violations (was 45), none new except a missing PWR_FLAG on
+3V3 now that the CH340C no longer drives it.

Co-Authored-By: Claude Opus 5.5 <noreply@anthropic.com>
Parts:
- D10: LCSC (none) -> C19077549
- D11: value DSS14U -> DSK16; LCSC (none) -> C22466351
- D9: value ESDCAN01-2BWY -> PESD2CAN; footprint Package_TO_SOT_SMD:SOT-323_SC-70 -> Package_TO_SOT_SMD:SOT-23; LCSC (none) -> C2687131
- F3: value 0ZCG0050AF2C -> 1812L050/60GR; footprint ESP32-PDM-BASE:0ZCG0050AF2C -> Fuse:Fuse_1812_4532Metric; LCSC (none) -> C19078719
- U5: LCSC (none) -> C2878225
- U6: LCSC (none) -> C37396819

Commit message: Harden inputs for 30 V, finish BOM swaps, clean up ERC
- Switch inputs R3/R4/R7/R8: 330 R -> 4.7k 1206. 2 mA at 10.5 V,
  6.1 mA / 0.18 W at 30 V. LTV-247 CTR >= 50 % at 5 mA, ~0.7x at 2 mA
  (datasheet fig. 10) -> >= 0.7 mA out vs 0.33 mA needed.
- D1: SMAJ30CA (clamp 48.4 V, below the 50 V input caps).
- D10: SMAJ18CA on NMEA 2000 NET-S (9-16 V); clamp 29.2 V protects the
  TPS7B91 (42 V abs max). SMAJ33CA clamped at 53 V.
- F2: SMD0805B050TF; D4-D6: PESD0402V05; J4: WJ15EDGVC-3.81-04P
  (MCV 1.5 clone, footprint kept - verify against datasheet).
- ERC: PWR_FLAGs on +3V3, GND, VBUS, buck VIN, CAN LDO input, GND_CAN;
  LMR51610 symbol CB/FB/SW pins passive; spare GPIOs no-connect;
  orphaned CH340 GND symbol and IO18 stub removed; LED_C stub wires
  trimmed to their labels.

Netlist connectivity identical to previous commit. ERC: 8 left, all
lib_symbol_mismatch (BC817, LTV-247) - use Update Symbols from Library.

Co-Authored-By: Claude Opus 5.5 <noreply@anthropic.com>
Parts:
- D10: value SMAJ33CA -> SMAJ18CA; LCSC C19077549 -> C19077539
- J4: value Conn_01x04 -> WJ15EDGVC-3.81-04P; LCSC (none) -> C8410
Changed lines of the file:
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@@
 			)
 		)
-		(property "Value" "SMAJ33CA"
+		(property "Value" "SMAJ18CA"
 			(at 148.59 54.6099 90)
 			(effects
@@
 			)
 		)
-		(property "LCSC" "C19077549"
+		(property "LCSC" "C19077539"
 			(at 146.05 53.34 0)
 			(effects
@@
 			)
 		)
-		(property "Value" "Conn_01x04"
+		(property "Value" "WJ15EDGVC-3.81-04P"
 			(at 187.96 99.0599 0)
 			(effects
@@
 			)
 		)
+		(property "LCSC" "C8410"
+			(at 185.42 96.52 0)
+			(effects
+				(font
+					(size 1.27 1.27)
+				)
+				(hide yes)
+			)
+		)
 		(pin "4"
 		)
@@
 					(unit 1)
 				)
+			)
+		)
+	)
+	(symbol
+		(lib_id "power:PWR_FLAG")
+		(at 124.46 66.04 0)
+		(unit 1)
+		(exclude_from_sim no)
+		(in_bom no)
+		(on_board yes)
+		(dnp no)
+		(fields_autoplaced yes)
+		(property "Reference" "#FLG03"
+			(at 127 64.77 0)
+			(effects
+				(font
+					(size 1.27 1.27)
+				)
+				(hide yes)
+			)
+		)
+		(property "Value" "PWR_FLAG"
+			(at 127 67.31 0)
+			(effects
+				(font
+					(size 1.27 1.27)
+				)
+				(justify left)
+			)
+		)
+		(property "Footprint" ""
+			(at 124.46 66.04 0)
+			(effects
+				(font
+					(size 1.27 1.27)
+				)
+				(hide yes)
+			)
+		)
+		(property "Datasheet" "~"
+			(at 124.46 66.04 0)
+			(effects
+				(font
+					(size 1.27 1.27)
+				)
+				(hide yes)
+			)
+		)
+		(property "Description" "Special symbol for telling ERC where power comes from"
+			(at 124.46 66.04 0)
+			(effects
+				(font
+					(size 1.27 1.27)
+				)
+				(hide yes)
+			)
+		)
+		(pin "1"
+		)
+		(instances
+			(project "ESP32-PDM-BASE"
+				(path "/d0898527-243c-48e9-a217-df57be741056/4abda9db-3578-40b6-8ca1-53f040286d67"
+					(reference "#FLG03")
+					(unit 1)
+				)
+			)
+		)
+	)
+	(symbol
+		(lib_id "power:PWR_FLAG")
+		(at 149.86 105.41 0)
+		(unit 1)
+		(exclude_from_sim no)
+		(in_bom no)
+		(on_board yes)
+		(dnp no)
+		(fields_autoplaced yes)
+		(property "Reference" "#FLG06"
+			(at 152.4 104.14 0)
+			(effects
+				(font
+					(size 1.27 1.27)
+				)
+				(hide yes)
+			)
+		)
+		(property "Value" "PWR_FLAG"
+			(at 152.4 106.68 0)
+			(effects
+				(font
+					(size 1.27 1.27)
+				)
+				(justify left)
+			)
+		)
+		(property "Footprint" ""
+			(at 149.86 105.41 0)
+			(effects
+				(font
+					(size 1.27 1.27)
+				)
+				(hide yes)
+			)
+		)
+		(property "Datasheet" "~"
+			(at 149.86 105.41 0)
+			(effects
+				(font
+					(size 1.27 1.27)
+				)
+				(hide yes)
+			)
+		)
+		(property "Description" "Special symbol for telling ERC where power comes from"
+			(at 149.86 105.41 0)
+			(effects
+				(font
+					(size 1.27 1.27)
+				)
+				(hide yes)
+			)
+		)
+		(pin "1"
+		)
+		(instances
+			(project "ESP32-PDM-BASE"
+				(path "/d0898527-243c-48e9-a217-df57be741056/4abda9db-3578-40b6-8ca1-53f040286d67"
+					(reference "#FLG06")
+					(unit 1)
+				)
