File: power-usb.kicad_sch (KiCad schematic)
At the start: 35 parts, among them J3 USB4145-03-0170-C, Q1 BC817-25LT1G, Q2 BC817-25LT1G, U3 LMR51610YDBVR, U4 CH340C

Commit message: Apply JLCPCB BOM audit fixes and add module ID / switch sense
- Remove CH340C and auto-reset circuit; USB-C goes to native USB
  (IO19 = D-, IO20 = D+). UART0 left unconnected.
- USB-C: HRO TYPE-C-31-M-12 (shell pins renumbered SH to match footprint).
- F1/F3: 1812L050/60GR (60 V, 500 mA hold); old part was rated 30 V max.
- D2/D3/D11: DSK16 (60 V) replacing out-of-stock DSS14U.
- D9: PESD2CAN replacing unavailable ESDCAN01-2BWY (SOT-23).
- L1: SWPA6045S8R2MT (Isat 3.9 A > LMR51610 peak limit 1.95 A).
- Feedback divider 68k/22k (basic parts): Vout 3.27 V with Vref 0.8 V.
- Basic-library swaps: TS-1187A buttons, 0805 2.2uF/50V, 49.9 R,
  BC817-40.
- Move the ST pull-ups to the output module.
- Header pin 12 becomes MOD_ID (IO1, 10k pull-up).
- SW1-SW4 to IO14/IO15/IO16/IO21 with 10k pull-downs, so the firmware
  can read the physical switches.
- Add LCSC part numbers for changed parts and main ICs.

ERC: 38 violations (was 45), none new except a missing PWR_FLAG on
+3V3 now that the CH340C no longer drives it.

Co-Authored-By: Claude Opus 5.5 <noreply@anthropic.com>
Parts:
- removed D7, D8: BAT54A, Package_TO_SOT_SMD:SOT-23, symbol Diode:BAT54A
- removed Q1, Q2: BC817-25LT1G, Package_TO_SOT_SMD:SOT-23-3, symbol Transistor_BJT:BC817
- removed R13, R14: 10k, Resistor_SMD:R_0402_1005Metric, symbol Device:R
- removed U4: CH340C, Package_SO:SOIC-16_3.9x9.9mm_P1.27mm, symbol Interface_USB:CH340C
- C1, C3: footprint Capacitor_SMD:C_0603_1608Metric -> Capacitor_SMD:C_0805_2012Metric; LCSC (none) -> C377773
- D1: LCSC (none) -> C19077549
- D2, D3: value DSS14U -> DSK16; LCSC (none) -> C22466351
- F1: value 0ZCG0050AF2C -> 1812L050/60GR; footprint ESP32-PDM-BASE:0ZCG0050AF2C -> Fuse:Fuse_1812_4532Metric; LCSC (none) -> C19078719
- J3: value USB4145-03-0170-C -> TYPE-C-31-M-12; footprint ESP32-PDM-BASE:GCT_USB4145-03-0170-C -> Connector_USB:USB_C_Receptacle_HRO_TYPE-C-31-M-12; LCSC (none) -> C165948
- L1: value VLS6045AF-8R2M -> SWPA6045S8R2MT; footprint ESP32-PDM-BASE:IND_VLS6045AF-8R2M -> Inductor_SMD:L_Sunlord_SWPA6045S; LCSC (none) -> C96963
- R10: value 22.1k -> 22k; LCSC (none) -> C31850
- R9: value 69.8k -> 68k; LCSC (none) -> C23231
- SW_BOOT1, SW_RESET1: footprint Button_Switch_SMD:SW_SPST_PTS647_Sx38 -> Button_Switch_SMD:SW_Push_1P1T_XKB_TS-1187A; LCSC (none) -> C318884
- U3: LCSC (none) -> C22427220
Connections:
- net BOOT: now also C7.2, SW_BOOT1.1
- net GND: now also J3.SH (SHIELD); no longer J3.S1 (SHIELD), J3.S2 (SHIELD), J3.S3 (SHIELD), J3.S4 (SHIELD)
- net RESET: now also C9.1, SW_RESET1.1
- net USB_DP: now reaches D5.2 (A2), J3.A6 (DP1), J3.B6 (DP2)
- net USB_DN: now reaches D6.2 (A2), J3.A7 (DN1), J3.B7 (DN2)
- no-connect marks 7 -> 2

Commit message: Harden inputs for 30 V, finish BOM swaps, clean up ERC
- Switch inputs R3/R4/R7/R8: 330 R -> 4.7k 1206. 2 mA at 10.5 V,
  6.1 mA / 0.18 W at 30 V. LTV-247 CTR >= 50 % at 5 mA, ~0.7x at 2 mA
  (datasheet fig. 10) -> >= 0.7 mA out vs 0.33 mA needed.
- D1: SMAJ30CA (clamp 48.4 V, below the 50 V input caps).
- D10: SMAJ18CA on NMEA 2000 NET-S (9-16 V); clamp 29.2 V protects the
  TPS7B91 (42 V abs max). SMAJ33CA clamped at 53 V.
- F2: SMD0805B050TF; D4-D6: PESD0402V05; J4: WJ15EDGVC-3.81-04P
  (MCV 1.5 clone, footprint kept - verify against datasheet).
- ERC: PWR_FLAGs on +3V3, GND, VBUS, buck VIN, CAN LDO input, GND_CAN;
  LMR51610 symbol CB/FB/SW pins passive; spare GPIOs no-connect;
  orphaned CH340 GND symbol and IO18 stub removed; LED_C stub wires
  trimmed to their labels.

Netlist connectivity identical to previous commit. ERC: 8 left, all
lib_symbol_mismatch (BC817, LTV-247) - use Update Symbols from Library.

Co-Authored-By: Claude Opus 5.5 <noreply@anthropic.com>
Parts:
- D1: value SMAJ33CA -> SMAJ30CA; LCSC C19077549 -> C19077548
- D4, D5, D6: value GG040205170N2P -> PESD0402V05; LCSC (none) -> C19626254
- F2: value 0ZCK0050FF2E -> SMD0805B050TF; footprint ESP32-PDM-BASE:0ZCK_BEL -> Fuse:Fuse_0805_2012Metric; LCSC (none) -> C269104
Changed lines of the file:
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@@
 			)
 		)
-		(property "Value" "GG040205170N2P"
+		(property "Value" "PESD0402V05"
 			(at 45.72 126.746 90)
 			(effects
@@
 		)
 		(property "Description" "Bidirectional transient-voltage-suppression diode"
+			(at 64.77 124.46 0)
+			(effects
+				(font
+					(size 1.27 1.27)
+				)
+				(hide yes)
+			)
+		)
+		(property "LCSC" "C19626254"
 			(at 64.77 124.46 0)
 			(effects
@@
 			)
 		)
-		(property "Value" "GG040205170N2P"
+		(property "Value" "PESD0402V05"
 			(at 90.17 80.0099 90)
 			(effects
@@
 		)
 		(property "Description" "Bidirectional transient-voltage-suppression diode"
+			(at 87.63 78.74 0)
+			(effects
+				(font
+					(size 1.27 1.27)
+				)
+				(hide yes)
+			)
+		)
+		(property "LCSC" "C19626254"
 			(at 87.63 78.74 0)
 			(effects
@@
 			)
 		)
-		(property "Value" "0ZCK0050FF2E"
+		(property "Value" "SMD0805B050TF"
 			(at 64.77 68.58 90)
 			(effects
@@
 			)
 		)
-		(property "Footprint" "ESP32-PDM-BASE:0ZCK_BEL"
+		(property "Footprint" "Fuse:Fuse_0805_2012Metric"
 			(at 69.85 71.12 0)
 			(effects
@@
 			)
 		)
+		(property "LCSC" "C269104"
+			(at 64.77 72.39 0)
+			(effects
+				(font
+					(size 1.27 1.27)
+				)
+				(hide yes)
+			)
+		)
 		(pin "2"
 		)
@@
 				(path "/d0898527-243c-48e9-a217-df57be741056/4e2a30d7-59a0-4ccb-98ec-adc6bcb9c0a2"
 					(reference "#PWR01")
-					(unit 1)
-				)
-			)
-		)
-	)
-	(symbol
-		(lib_id "power:GND")
-		(at 106.68 165.1 0)
-		(unit 1)
-		(exclude_from_sim no)
-		(in_bom yes)
-		(on_board yes)
-		(dnp no)
-		(fields_autoplaced yes)
-		(property "Reference" "#PWR011"
-			(at 106.68 171.45 0)
-			(effects
-				(font
-					(size 1.27 1.27)
-				)
-				(hide yes)
-			)
-		)
-		(property "Value" "GND"
-			(at 106.68 170.18 0)
-			(effects
-				(font
-					(size 1.27 1.27)
-				)
-			)
-		)
-		(property "Footprint" ""
-			(at 106.68 165.1 0)
-			(effects
-				(font
-					(size 1.27 1.27)
-				)
-				(hide yes)
-			)
-		)
-		(property "Datasheet" ""
-			(at 106.68 165.1 0)
-			(effects
-				(font
-					(size 1.27 1.27)
-				)
-				(hide yes)
-			)
-		)
-		(property "Description" "Power symbol creates a global label with name \"GND\" , ground"
-			(at 106.68 165.1 0)
-			(effects
-				(font
-					(size 1.27 1.27)
-				)
-				(hide yes)
-			)
-		)
-		(pin "1"
-		)
-		(instances
-			(project "ESP32-PDM-BASE"
-				(path "/d0898527-243c-48e9-a217-df57be741056/4e2a30d7-59a0-4ccb-98ec-adc6bcb9c0a2"
-					(reference "#PWR011")
 					(unit 1)
 				)
@@
 			)
 		)
-		(property "Value" "GG040205170N2P"
+		(property "Value" "PESD0402V05"
 			(at 72.39 125.7299 90)
 			(effects
@@
 		)
 		(property "Description" "Bidirectional transient-voltage-suppression diode"
+			(at 69.85 124.46 0)
+			(effects
+				(font
+					(size 1.27 1.27)
+				)
+				(hide yes)
+			)
+		)
+		(property "LCSC" "C19626254"
 			(at 69.85 124.46 0)
 			(effects
@@
 			)
 		)
-		(property "Value" "SMAJ33CA"
+		(property "Value" "SMAJ30CA"
 			(at 91.44 45.7199 90)
 			(effects
@@
 			)
 		)
-		(property "LCSC" "C19077549"
+		(property "LCSC" "C19077548"
 			(at 88.9 44.45 0)
 			(effects
@@
 		)
 	)
+	(symbol
+		(lib_id "power:PWR_FLAG")
+		(at 22.86 83.82 0)
+		(unit 1)
+		(exclude_from_sim no)
+		(in_bom no)
+		(on_board yes)
+		(dnp no)
+		(fields_autoplaced yes)
+		(property "Reference" "#FLG01"
+			(at 25.4 82.55 0)
+			(effects
+				(font
+					(size 1.27 1.27)
+				)
+				(hide yes)
+			)
+		)
+		(property "Value" "PWR_FLAG"
+			(at 25.4 85.09 0)
+			(effects
+				(font
+					(size 1.27 1.27)
+				)
+				(justify left)
+			)
+		)
+		(property "Footprint" ""
+			(at 22.86 83.82 0)
+			(effects
+				(font
+					(size 1.27 1.27)
+				)
+				(hide yes)
+			)
+		)
+		(property "Datasheet" "~"
+			(at 22.86 83.82 0)
+			(effects
+				(font
+					(size 1.27 1.27)
+				)
+				(hide yes)
+			)
+		)
+		(property "Description" "Special symbol for telling ERC where power comes from"
+			(at 22.86 83.82 0)
+			(effects
+				(font
+					(size 1.27 1.27)
+				)
+				(hide yes)
+			)
+		)
+		(pin "1"
+		)
+		(instances
+			(project "ESP32-PDM-BASE"
+				(path "/d0898527-243c-48e9-a217-df57be741056/4e2a30d7-59a0-4ccb-98ec-adc6bcb9c0a2"
+					(reference "#FLG01")
+					(unit 1)
+				)
+			)
+		)
+	)
+	(symbol
+		(lib_id "power:PWR_FLAG")
+		(at 163.83 68.58 0)
+		(unit 1)
+		(exclude_from_sim no)
+		(in_bom no)
+		(on_board yes)
+		(dnp no)
+		(fields_autoplaced yes)
+		(property "Reference" "#FLG02"
+			(at 166.37 67.31 0)
+			(effects
+				(font
+					(size 1.27 1.27)
+				)
+				(hide yes)
+			)
+		)
+		(property "Value" "PWR_FLAG"
+			(at 166.37 69.85 0)
+			(effects
+				(font
+					(size 1.27 1.27)
+				)
+				(justify left)
+			)
+		)
+		(property "Footprint" ""
+			(at 163.83 68.58 0)
+			(effects
+				(font
+					(size 1.27 1.27)
+				)
+				(hide yes)
+			)
+		)
+		(property "Datasheet" "~"
+			(at 163.83 68.58 0)
+			(effects
+				(font
+					(size 1.27 1.27)
+				)
+				(hide yes)
+			)
+		)
+		(property "Description" "Special symbol for telling ERC where power comes from"
+			(at 163.83 68.58 0)
+			(effects
+				(font
+					(size 1.27 1.27)
+				)
+				(hide yes)
+			)
+		)
+		(pin "1"
+		)
+		(instances
+			(project "ESP32-PDM-BASE"
+				(path "/d0898527-243c-48e9-a217-df57be741056/4e2a30d7-59a0-4ccb-98ec-adc6bcb9c0a2"
+					(reference "#FLG02")
+					(unit 1)
+				)
+			)
+		)
+	)
